File: pcb/moisture.kicad_pcb (KiCad board)
At the start: 2 copper layers, 33 parts

Commit message: Update pcb design
Parts:
- removed the REF** at (68.6, 120.7)
- added ?: , , F.Cu at (73.7, 120.7)
- added ?: , , F.Cu at (71.1, 120.7)
- added ?: , , F.Cu at (76.2, 120.7)
- added ?: , , F.Cu at (68.6, 120.7)
